Commit message: synapses

File: body.urdf (robot description, URDF)
Before this commit: robot robot, 3 links, 2 joints
Joints:
- removed joint Torso_Leg
- removed joint Torso_Leg2
- added joint Torso_backLeg: type revolute, parent Torso, child backLeg, origin xyz=-.5 0 1 rpy=0 0 0, axis 0 1 0, limit lower=-3.14159 upper=3.14159 effort=0.0 velocity=0.0
- added joint Torso_frontLeg: type revolute, parent Torso, child frontLeg, origin xyz=.5 0 1 rpy=0 0 0, axis 0 1 0, limit lower=-3.14159 upper=3.14159 effort=0.0 velocity=0.0

Commit message: Cleanup..
* Switch exists for toggling hidden neuron or original synapse configuration
* Some code added to plot the results of different iterations

File: body.urdf (robot description, URDF)
Before this commit: robot robot, 3 links, 2 joints
Links:
- added link backFoot, mass 1; collision box size=0.2 0.2 1; visual box size=0.2 0.2 1
- added link frontFoot, mass 1; collision box size=0.2 0.2 1; visual box size=0.2 0.2 1
- added link leftFoot, mass 1; collision box size=0.2 0.2 1; visual box size=0.2 0.2 1
- added link leftLeg, mass 1; collision box size=1 0.2 0.2; visual box size=1 0.2 0.2
- added link rightFoot, mass 1; collision box size=0.2 0.2 1; visual box size=0.2 0.2 1
- added link rightLeg, mass 1; collision box size=1 0.2 0.2; visual box size=1 0.2 0.2
- link backLeg: geometry collision box size=0.2 1 0.2; visual box size=0.2 1 0.2
- link frontLeg: geometry collision box size=0.2 1 0.2; visual box size=0.2 1 0.2
Joints:
- added joint Torso_leftLeg: type revolute, parent Torso, child leftLeg, origin xyz=-.5 0 1.5 rpy=0 0 0, axis 0 1 0, limit lower=-3.14159 upper=3.14159 effort=0.0 velocity=0.0
- added joint Torso_rightLeg: type revolute, parent Torso, child rightLeg, origin xyz=.5 0 1.5 rpy=0 0 0, axis 0 1 0, limit lower=-3.14159 upper=3.14159 effort=0.0 velocity=0.0
- added joint backLeg_backFoot: type revolute, parent backLeg, child backFoot, origin xyz=0 -1 0 rpy=0 0 0, axis 1 0 0, limit lower=-3.14159 upper=3.14159 effort=0.0 velocity=0.0
- added joint frontLeg_frontFoot: type revolute, parent frontLeg, child frontFoot, origin xyz=0 1 0 rpy=0 0 0, axis 1 0 0, limit lower=-3.14159 upper=3.14159 effort=0.0 velocity=0.0
- added joint leftLeg_leftFoot: type revolute, parent leftLeg, child leftFoot, origin xyz=-1 0 0 rpy=0 0 0, axis 0 1 0, limit lower=-3.14159 upper=3.14159 effort=0.0 velocity=0.0
- added joint rightLeg_rightFoot: type revolute, parent rightLeg, child rightFoot, origin xyz=1 0 0 rpy=0 0 0, axis 0 1 0, limit lower=-3.14159 upper=3.14159 effort=0.0 velocity=0.0
- joint Torso_backLeg: axis 0 1 0 -> 1 0 0; origin xyz=-.5 0 1 rpy=0 0 0 -> xyz=0 -0.5 1.5 rpy=0 0 0
- joint Torso_frontLeg: axis 0 1 0 -> 1 0 0; origin xyz=.5 0 1 rpy=0 0 0 -> xyz=0 .5 1.5 rpy=0 0 0
